Commit message: Update rabbit cube & make aprilcube larger

File: urdf/rabbit.urdf (robot description, URDF)
Before this commit: robot rabbit, 1 links, 0 joints
Links:
- removed link rabbit_sphere
- added link rabbit_cube, mass 1.0; visual box size=2 2 2

Commit message: Update rabbit waypoints

File: urdf/rabbit.urdf (robot description, URDF)
Before this commit: robot rabbit, 1 links, 0 joints
Links:
- link rabbit_cube: geometry visual box size=1 1 1
