Commit message: Updated sandwich.launch with functional april_cube rabbit model

File: urdf/april_cube.xacro (robot description, xacro)
@@ -23,5 +23,5 @@
       </inertial>
       <visual>
-        <material name="white" />
+        <material name="White" />
         <origin xyz="0 0 0" />
         <geometry>
@@ -45,6 +45,6 @@
       <kp>1000000.0</kp>
       <kd>1.0</kd>
-    </gazebo>
-    <!-- top -->
+  </gazebo>
+  <!-- top -->
     <xacro:apriltag_marker namespace="" name="${name}_tag_${id_top}" parent="${name}"
            family="36h11" ID="${id_top}" size="${marker_size}">

File: urdf/april_cube_demo.xacro (robot description, xacro)
@@ -10,38 +10,14 @@
        in this case.
   -->
-  <link name="world" />
-  <link name="doro/world" />
-  <joint name="hugo" type="fixed">
+  <xacro:april_cube name="april_cube" size="1.5" marker_size="1.25"
+      id_top="0" id_front="1" id_right="2" id_back="3" id_left="4" id_bottom="5" />
+  <!--link name="world" />
+  <joint name="april_cube_joint" type="fixed" >
     <parent link="world" />
-    <child  link="doro/world" />
-    <origin xyz="0 0 1" rpy="0 0 0" />
+    <child  link="april_cube" />
+    <origin xyz="0 0 0" rpy=" 0 0 0" />
   </joint>
-  <xacro:april_cube name="april_cube_60" size="1.1" marker_size="1"
-      id_top="60" id_front="61" id_right="62" id_back="63" id_left="64" id_bottom="65" />
-  <joint name="april_cube_60_joint" type="fixed" >
-    <parent link="world" />
-    <child  link="april_cube_60" />
-    <origin xyz="1 0 0.1" rpy=" 0 0 0" />
-  </joint>
-  <!--xacro:april_cube name="april_cube_40" size="0.071" marker_size="0.07"
-      id_top="40" id_front="41" id_right="42" id_back="43" id_left="44" id_bottom="45" />
-  <joint name="april_cube_40_joint" type="fixed" >
-    <parent link="world" />
-    <child  link="april_cube_40" />
-    <origin xyz="0 0 0.1" rpy=" 0 0 0" />
-  </joint>
-  <xacro:april_cube name="april_cube_46" size="0.071" marker_size="0.07"
-      id_top="46" id_front="47" id_right="48" id_back="49" id_left="50" id_bottom="51" />
-  <joint name="april_cube_46_joint" type="fixed" >
-    <parent link="world" />
-    <child  link="april_cube_46" />
-    <origin xyz="0.3 0 0.1" rpy=" 0 0 0" />
-  </joint>
-  <xacro:april_cube name="april_cube_52" size="0.071" marker_size="0.07"
-      id_top="52" id_front="53" id_right="54" id_back="55" id_left="56" id_bottom="57" />
-  <joint name="april_cube_52_joint" type="fixed" >
-    <parent link="world" />
-    <child  link="april_cube_52" />
-    <origin xyz="0.6 0 0.1" rpy=" 0 0 0" />
-  </joint-->
+  <gazebo reference="april_cube_joint">
+    <preserveFixedJoint>true</preserveFixedJoint>
+  </gazebo-->
 </robot>
