Commit message: Boat follow updates

File: urdf/sandwich.xacro (robot description, xacro)
@@ -75,21 +75,21 @@
 	<!-- front -->
     <xacro:apriltag_marker namespace="$(arg namespace)" name="/tag_0" parent="/base_link"
-           family="36h11" ID="10" size="0.625">
-           <origin xyz="0 0 1.5" rpy="1.571 0 1.571" />
+           family="36h11" ID="10" size="1.25">
+           <origin xyz="0 0 2" rpy="1.571 0 1.571" />
     </xacro:apriltag_marker>
     <!-- back -->
     <xacro:apriltag_marker namespace="$(arg namespace)" name="/tag_1" parent="/base_link"
-           family="36h11" ID="11" size="0.625">
-           <origin xyz="-3.8 0 1.5" rpy="1.571 0 -1.571" />
+           family="36h11" ID="11" size="1.25">
+           <origin xyz="-3.8 0 2" rpy="1.571 0 -1.571" />
     </xacro:apriltag_marker>
   <!-- left -->
     <xacro:apriltag_marker namespace="$(arg namespace)" name="/tag_2" parent="/base_link"
-           family="36h11" ID="12" size="0.625">
-           <origin xyz="-1 0.7 1.5" rpy="1.571 3.141 3.141" />
+           family="36h11" ID="12" size="1.25">
+           <origin xyz="-1 0.7 2" rpy="1.571 3.141 3.141" />
     </xacro:apriltag_marker>
     <!-- right -->
     <xacro:apriltag_marker namespace="$(arg namespace)" name="/tag_3" parent="/base_link"
-           family="36h11" ID="13" size="0.625">
-           <origin xyz="-1.0 -0.7 1.5" rpy="1.571 3.141 0" />
+           family="36h11" ID="13" size="1.25">
+           <origin xyz="-1.0 -0.7 2" rpy="1.571 3.141 0" />
     </xacro:apriltag_marker>
 </robot>

Commit message: Add p3d, update vbap and multi_follow

File: urdf/sandwich.xacro (robot description, xacro)
@@ -52,10 +52,19 @@
   </xacro:if>
   <!-- Sensors -->
+   <gazebo>
+    <plugin name="p3d_plugin_sandwich" filename="libgazebo_ros_p3d.so">
+      <bodyName>$(arg namespace)/base_link</bodyName>
+      <frameName>world</frameName>
+      <updateRate>10.0</updateRate>
+      <topicName>$(arg namespace)/sensors/p3d</topicName>
+      <xyzOffset>0 0 0</xyzOffset>
+      <rpyOffset>0 0 0</rpyOffset>
+      <gaussianNoise>0</gaussianNoise>
+    </plugin>
+  </gazebo>
   <xacro:arg name="camera_namespace" default="cameras/"/>
   <xacro:arg name="sensor_namespace" default="sensors/"/>
-  <xacro:arg name="pinger_namespace" default="pingers/"/>
   <xacro:property name="camera_namespace" value="$(arg camera_namespace)" scope="global" />
   <xacro:property name="sensor_namespace" value="$(arg sensor_namespace)" scope="global" />
-  <xacro:property name="pinger_namespace" value="$(arg pinger_namespace)" scope="global" />
   <xacro:wamv_camera name="front_left_camera"  x="3.8" y="0.25"  z="1.3"
   post_z_from="1.1" P="${radians(0)}" Y="${radians(10)}" />
@@ -72,8 +81,4 @@
   <xacro:lidar name="front_lidar" type="16_beam" x="3.9" z="1.4"
   P="${radians(8)}" post_z_from="1.1"/>
-  <xacro:wamv_gps name="gps" x="-1.0" z="1.28"
-  	update_rate="20" />
-  <xacro:wamv_imu name="imu" y="-0.2" z="1.0" update_rate="100" />
-  <xacro:wamv_pinger name="pinger" frameId="$(arg namespace)/pinger" />
 	<!--AprilTags-->
 	<!-- front -->
