Commit message: Rabbit follow mod; boat dynamics improvements

File: urdf/sandwich.urdf.xacro (robot description, xacro)
@@ -29,38 +29,2 @@
 	</xacro:macro>
 </robot>
-<!-- <?xml version="1.0"?> -->
-<!-- <robot xmlns:xacro="http://ros.org/wiki/xacro" name="sandwich"> -->
-	<!-- <xacro:property name="namespace" default="sandwich"/> -->
-	<!-- <xacro:macro name="sandwich_robot" params="namespace"> -->
-		<!-- "Dummy" base link to eliminate root link inertia warning -->
-		<!-- <link name="sandwich/base_link"/> -->
-		<!-- Main link -->
-		<!-- <link name="sandwich/sandwich_link">
-			<inertial>
-				<origin xyz="0 0 0" rpy="0 0 0"/>
-				<mass value="2"/>
-				<inertia
-					ixx="5.0" ixy="0.0" ixz="0.0"
-					iyy="3.6" iyz="0.0"
-					izz="1.7"/>
-			</inertial>
-			<visual>
-				<origin xyz="0 0 0" rpy="0 0 0"/>
-				<geometry>
-					<mesh filename="file://$(find sandwich_description)/models/sandwich_base/sandwich.dae" scale="1 1 1"/>
-				</geometry>
-			</visual>
-			<collision>
-				<origin xyz="0 0 0" rpy="0 0 0"/>
-				<geometry>
-					<mesh filename="file://$(find sandwich_description)/models/sandwich_base/sandwich.dae" scale="1 1 1"/>
-				</geometry>
-			</collision>
-		</link>
-		<joint name="sandwich/sandwich_base_joint" type="fixed">
-			<origin xyz="0 0 0" rpy="0 0 0"/>
-			<parent link="sandwich/base_link"/>
-			<child link="sandwich/sandwich_link"/>
-		</joint> -->
-	<!-- </xacro:macro> -->
-<!-- </robot> -->

File: urdf/sandwich.xacro (robot description, xacro)
@@ -8,5 +8,5 @@
   <xacro:arg name="right_ID" default="13"/>
   <!-- Include macros for dynamics plugins -->
-  <xacro:include filename="$(find sandwich_description)/urdf/macros.xacro" />
+  <xacro:include filename="$(find optical_swarm)/urdf/macros.xacro" />
   <!-- Attach hydrodynamics plugin -->
   <xacro:usv_dynamics_gazebo name="sandwich_dynamics_plugin" namespace="$(arg namespace)"/>

File: urdf/thrusters.xacro (robot description, xacro)
@@ -90,5 +90,5 @@
         <cmdTimeout>1.0</cmdTimeout>
         <robotNamespace>${namespace}</robotNamespace>
-        <xacro:include filename="$(find sandwich_description)/urdf/sandwich_thruster_config.xacro" />
+        <xacro:include filename="$(find optical_swarm)/urdf/sandwich_thruster_config.xacro" />
         <!-- Angle must be disabled for VORC -->
         <xacro:sandwich_thruster_config name="left"/>
