Commit message: Speed lookup updates

File: urdf/sandwich_dynamics_plugin.xacro (robot description, xacro)
@@ -10,5 +10,5 @@
         <waterDensity>1024.0</waterDensity>
         <!-- Added mass -->
-        <xDotU>0</xDotU>
+        <xDotU>1000</xDotU>
         <yDotV>26000</yDotV>
         <zDotW>31000</zDotW>
@@ -17,8 +17,8 @@
         <nDotR>0.0</nDotR>
         <!-- Linear and quadratic drag -->
-        <xU>500.0</xU>
-        <xUU>500.0</xUU>
-        <yV>240.0</yV>
-        <yVV>2600</yVV>
+        <xU>300.0</xU>
+        <xUU>3000.0</xUU>
+        <yV>1200.0</yV>
+        <yVV>12000</yVV>
         <zW>50000.0</zW>
         <zWW>0.0</zWW>
@@ -27,6 +27,6 @@
         <mQ>500000.0</mQ>
         <mQQ>5000.0</mQQ>
-        <nR>350000.0</nR>
-        <nRR>0.0</nRR>
+        <nR>550000.0</nR>
+        <nRR>5000.0</nRR>
         <!-- General dimensions -->
         <!--<boatArea>2.2</boatArea>-->

File: urdf/sandwich_thruster_config.xacro (robot description, xacro)
@@ -13,6 +13,6 @@
 			<mappingType>0</mappingType>
 			<maxCmd>1.0</maxCmd>
-			<maxForceFwd>65000.0</maxForceFwd>
-			<maxForceRev>-65000.0</maxForceRev>
+			<maxForceFwd>145000.0</maxForceFwd>
+			<maxForceRev>-145000.0</maxForceRev>
 			<maxAngle>${pi/2}</maxAngle>
 		</thruster>

File: urdf/thrusters.xacro (robot description, xacro)
@@ -31,5 +31,5 @@
     <joint name="left_chasis_engine_joint" type="revolute">
       <axis xyz="1 0 0"/>
-      <origin rpy="0 0 0" xyz="-3.8 1.5 0.285"/>
+      <origin rpy="0 0 0" xyz="-3.8 1.0 0.285"/>
       <parent link="${namespace}/base_link"/>
       <child link="left_engine_link"/>
@@ -73,5 +73,5 @@
     <joint name="right_chasis_engine_joint" type="revolute">
       <axis xyz="1 0 0"/>
-      <origin rpy="0 0 0" xyz="-3.8 -1.5 0.285"/>
+      <origin rpy="0 0 0" xyz="-3.8 -1.0 0.285"/>
       <parent link="${namespace}/base_link"/>
       <child link="right_engine_link"/>
